File: variations/Camden/V0.2.2/software/KiCad/Cell_Balancer/Cell_Balancer.kicad_pcb (KiCad board)
At the start: 2 copper layers, 45 x 70.5 mm, 13 parts, among them J1 Screw_Terminal_01x11

Commit message: added some identifiers to the pcb
Other:
- board text added: "Cell Balancer, V.0.2.2, 7/9/2026, Cebastione Bailey, University of South Carolina, ARTS Lab"
Changed lines of the file:
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@@
 		(layer "Edge.Cuts")
+	)
+	(gr_text "Cell Balancer, V.0.2.2, 7/9/2026, Cebastione Bailey,\n University of South Carolina, ARTS Lab"
+		(at 106.5 76 270)
+		(layer "F.SilkS")
+		(effects
+			(font
+				(size 1 1)
+				(thickness 0.1)
+			)
+			(justify left bottom)
+		)
 	)
 	(segment
